File: CoryDora.kicad_pcb (KiCad board)
At the start: 2 copper layers, 21 parts, among them J1 OLED_128x32, SW1 RotaryEncoder_Switch, U1 RP2040_Zero

Commit message: chore: complete layout in PCB editor
Parts:
- D1, D2, D3, D4, D5, D6, D7, D8, D9, U1: moved to B.Cu
- S2, S3, S4, S5, S6, S7, S8: footprint ScottoKeebs_Hotswap:Hotswap_MX_Plated -> ScottoKeebs_Hotswap:Hotswap_MX_Plated_1.00u
- S9: footprint ScottoKeebs_MX:MX_PCB_1.00u -> ScottoKeebs_Hotswap:Hotswap_MX_Plated_1.00u
- moved S7 108.6 mm to (134.6, 134.0), turned to 180 degrees
- moved S8 95.7 mm to (115.6, 134.0), turned to 180 degrees
- moved S5 89.7 mm to (115.6, 115.0), turned to 180 degrees
- moved SW1 85.4 mm to (147.4, 131.5)
- moved S1 84.6 mm to (134.6, 96.0), turned to 180 degrees
- moved D7 81.4 mm to (143.1, 124.1), turned to -90 degrees
- moved S4 79.8 mm to (134.6, 115.0), turned to 180 degrees
- moved J1 78.2 mm to (149.6, 125.0), turned to 90 degrees
- moved S6 78.0 mm to (96.6, 115.0), turned to 180 degrees
- moved D4 77.0 mm to (143.1, 106.3), turned to -90 degrees
- moved D1 72.4 mm to (143.1, 87.3), turned to -90 degrees
- moved S3 71.0 mm to (96.6, 96.0), turned to 180 degrees
- moved D8 67.8 mm to (125.6, 126.2), turned to -90 degrees
- moved U1 67.5 mm to (155.6, 98.0), turned to 180 degrees
- moved S9 65.6 mm to (96.6, 134.0), turned to 180 degrees
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Routing:
- net COLUMN2: track 0.00 -> 104.3 mm
- net COLUMN1: track 0.00 -> 83.9 mm
- net ROW2: track 0.00 -> 73.4 mm, vias 0 -> 1
- net ROW0: track 0.00 -> 68.0 mm
- net GND: track 0.00 -> 63.1 mm, vias 0 -> 2
- net ROW1: track 0.00 -> 61.2 mm, vias 0 -> 1
- net COLUMN0: track 0.00 -> 60.9 mm
- net MCU_5V: track 0.00 -> 44.4 mm, vias 0 -> 2
- net ENCODER_SW: track 0.00 -> 43.3 mm
- net ENCODER_B: track 0.00 -> 42.8 mm, vias 0 -> 1
- net OLED_SDA: track 0.00 -> 37.1 mm, vias 0 -> 2
- net ENCODER_A: track 0.00 -> 36.9 mm
- net OLED_SCL: track 0.00 -> 31.1 mm
- net Net-(D7-A): track 0.00 -> 15.9 mm
- net Net-(D9-A): track 0.00 -> 14.7 mm
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
Commit message: chore: completed PCB design
Parts:
- added H1: MountingHole, MountingHole:MountingHole_2.2mm_M2, F.Cu at (166.4, 142.4)
- added H2: MountingHole, MountingHole:MountingHole_2.2mm_M2, F.Cu at (168.1, 88.4)
- added H3: MountingHole, MountingHole:MountingHole_2.2mm_M2, F.Cu at (84.3, 88.9)
- added H4: MountingHole, MountingHole:MountingHole_2.2mm_M2, F.Cu at (84.2, 142.8)
Routing:
- net Net-(D4-A): track 14.7 -> 16.0 mm
Other:
- board outline added: 89.6 x 60.1 mm
