File: CoryDora.kicad_pcb (KiCad board)
At the start: 2 copper layers, 89.6 x 60.1 mm, 25 parts, among them J1 OLED_128x32, SW1 RotaryEncoder_Switch, U1 RP2040_Zero

Commit message: chore: added text and graphics to silkscreen
Parts:
- added G***: LOGO, Downloads:12, F.Cu at (165.6, 116.2)
Other:
- board text added: "CoryDora v1"
