File: CoryDora.kicad_sch (KiCad schematic)
At the start: 21 parts, among them J1 OLED_128x32, SW1 RotaryEncoder_Switch, U1 RP2040_Zero

Commit message: chore: completed PCB design
Parts:
- added H1, H2, H3, H4: MountingHole, MountingHole:MountingHole_2.2mm_M2, symbol Mechanical:MountingHole
